File: hw/layouts/pd12v6_manual/pd12v6_manual.kicad_pcb (KiCad board)
At the start: 4 copper layers, 40 x 32 mm, 31 parts

Commit message: pd12v6: correct USB-C 3D model position, U2 pin-1 dot, 5 A label
- EasyEDA's TYPE-C-31-M-12 model sits 2.31 mm behind its own footprint
  (pins behind the pads, mouth inside the edge). KiCad's footprint for the
  same part confirms our copper; KiCad has no 3D model for it, so offset
  the EasyEDA model instead. Mouth now overhangs the edge by 0.9 mm.
- U2 pin-1 dot was by pin 5; moved to pin 1 (bottom-right).
- Title silk said 4.5 A (old current-limited design); now 5 A.

Co-Authored-By: Claude Opus 5.5 <noreply@anthropic.com>
Other:
- board text added: "USB-C PD -> 12.6 V 5 A"
- board text removed: "USB-C PD -> 12.6 V 4.5 A"
Changed lines of the file:
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@@
 		(model "${KIPRJMOD}/../../parts/UNKNOWN_TYPE_C_31_M_12/USB-C_SMD-TYPE-C-31-M-12.step"
 			(offset
-				(xyz 0 0 0.85)
+				(xyz 0 -2.31 0.85)
 			)
 			(scale
@@
 	)
 	(gr_circle
-		(center 19 14.4)
-		(end 19.2 14.4)
+		(center 18.6 20.1)
+		(end 18.8 20.1)
 		(stroke
 			(width 0.15)
@@
 		(layer "Edge.Cuts")
 	)
-	(gr_text "USB-C PD -> 12.6 V 4.5 A"
+	(gr_text "USB-C PD -> 12.6 V 5 A"
 		(at 14 28 0)
 		(layer "F.SilkS")
@@
 	)
 	(zone
-		(net 17)
-		(net_name "VOUT")
+		(net 7)
+		(net_name "VBUS")
 		(layer "In2.Cu")
 		(hatch edge 0.5)
@@
 		(polygon
 			(pts
-				(xy 20.5 2) (xy 38.5 2) (xy 38.5 30) (xy 20.5 30)
+				(xy 7 2) (xy 19.9 2) (xy 19.9 24) (xy 7 24)
 			)
 		)
 	)
 	(zone
-		(net 7)
-		(net_name "VBUS")
+		(net 17)
+		(net_name "VOUT")
 		(layer "In2.Cu")
 		(hatch edge 0.5)
@@
 		(polygon
 			(pts
-				(xy 7 2) (xy 19.9 2) (xy 19.9 24) (xy 7 24)
+				(xy 20.5 2) (xy 38.5 2) (xy 38.5 30) (xy 20.5 30)
 			)
 		)
