File: hw/layouts/blind-io/controller-test/controller-test.kicad_pcb (KiCad board)
At the start: 2 copper layers, 36 parts

Commit message: Integrate motor supervision and add charger and Thread evaluation captures
Parts:
- removed C7: , blind-control-io:C0402
- removed R17, R18: , UNI_ROYAL_0402WGF1002TCE:R0402
- C2: footprint blind-control-io:C0805 -> blind-power:C0805
- SW1, SW2: footprint blind-control-io:SW-SMD_L3.9-W3.0-P4.45 -> blind-control-io:SW-SMD_4P-L3.5-W3.0-P1.6-LS4.6
Connections:
- SW1 pad 2: lv -> controller-1
- SW2 pad 2: lv -> controller-1-1
