File: hw/schematics/blind-controller/motor-test.kicad_sch (KiCad schematic)
At the start: 14 parts, among them U1 DRV8874PWPR

Commit message: Integrate motor supervision and add charger and Thread evaluation captures
Other:
- moved on the sheet: C1
