File: hw/layouts/blind-charger/charger-test/charger-test.kicad_pcb (KiCad board)
At the start: 2 copper layers, 35 parts

Commit message: Capture charger and logic supply with physical-pin and capacitor checks
Parts:
- added C22: , SAMSUNG_CL31A106KBHNNNE:C1206, F.Cu at (0.00, 0.00)
Changed lines of the file:
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@@
+		)
+	)
+	(footprint "SAMSUNG_CL31A106KBHNNNE:C1206"
+		(layer "F.Cu")
+		(at 0 0 0)
+		(property "Reference" "C22"
+			(at -2.66 0 0)
+			(layer "F.SilkS")
+			(hide yes)
+			(effects
+				(font
+					(size 1 1)
+					(thickness 0.15)
+				)
+				(justify right)
+			)
+		)
+		(property "Value" ""
+			(at 0 4)
+			(layer "F.Fab")
+			(effects
+				(font
+					(size 1 1)
+					(thickness 0.15)
+				)
+			)
+		)
+		(property "LCSC" "C13585"
+			(at 0 0 0)
+			(layer "User.9")
+			(hide yes)
+		)
+		(property "Manufacturer" "SAMSUNG"
+			(at 0 0 0)
+			(layer "User.9")
+			(hide yes)
+		)
+		(property "Partnumber" "CL31A106KBHNNNE"
+			(at 0 0 0)
+			(layer "User.9")
+			(hide yes)
+		)
+		(property "atopile_address" "charger.c_pmid4"
+			(at 0 0 0)
+			(layer "User.9")
+			(hide yes)
+		)
+		(property "lcsc_id" "C13585"
+			(at 0 0 0)
+			(layer "User.9")
+			(hide yes)
+		)
+		(attr smd)
+		(fp_line
+			(start 2.41 -1.09)
+			(end 0.93 -1.09)
+			(stroke
+				(width 0.15)
+				(type solid)
+			)
+			(layer "F.SilkS")
+			(layers "F.SilkS")
+			(locked no)
+		)
+		(fp_line
+			(start 0.93 1.09)
+			(end 2.41 1.09)
+			(stroke
+				(width 0.15)
+				(type solid)
+			)
+			(layer "F.SilkS")
+			(layers "F.SilkS")
+			(locked no)
+		)
+		(fp_line
+			(start 2.56 0.94)
+			(end 2.56 -0.94)
+			(stroke
+				(width 0.15)
+				(type solid)
+			)
+			(layer "F.SilkS")
+			(layers "F.SilkS")
+			(locked no)
+		)
+		(fp_line
+			(start -2.41 -1.09)
+			(end -0.93 -1.09)
+			(stroke
+				(width 0.15)
+				(type solid)
+			)
+			(layer "F.SilkS")
+			(layers "F.SilkS")
+			(locked no)
+		)
+		(fp_line
+			(start -0.93 1.09)
+			(end -2.41 1.09)
+			(stroke
+				(width 0.15)
+				(type solid)
+			)
+			(layer "F.SilkS")
+			(layers "F.SilkS")
+			(locked no)
+		)
+		(fp_line
+			(start -2.56 0.94)
+			(end -2.56 -0.94)
+			(stroke
+				(width 0.15)
+				(type solid)
+			)
+			(layer "F.SilkS")
+			(layers "F.SilkS")
+			(locked no)
+		)
+		(fp_arc
+			(start 2.56 0.94)
+			(mid 2.516066 1.046066)
+			(end 2.41 1.09)
+			(stroke
+				(width 0.15)
+				(type solid)
+			)
+			(layer "F.SilkS")
+			(locked no)
+		)
+		(fp_arc
+			(start 2.41 -1.09)
+			(mid 2.516066 -1.046066)
+			(end 2.56 -0.94)
+			(stroke
+				(width 0.15)
+				(type solid)
+			)
+			(layer "F.SilkS")
+			(locked no)
+		)
+		(fp_arc
+			(start -2.56 0.94)
+			(mid -2.516066 1.046066)
+			(end -2.41 1.09)
+			(stroke
+				(width 0.15)
+				(type solid)
+			)
+			(layer "F.SilkS")
+			(locked no)
+		)
+		(fp_arc
+			(start -2.41 -1.09)
+			(mid -2.516066 -1.046066)
+			(end -2.56 -0.94)
+			(stroke
+				(width 0.15)
+				(type solid)
+			)
+			(layer "F.SilkS")
+			(locked no)
+		)
+		(fp_circle
+			(center -1.6 0.8)
+			(end -1.57 0.8)
+			(stroke
+				(width 0.06)
+				(type solid)
+			)
+			(layer "F.Fab")
+			(locked no)
+		)
+		(pad "2" smd rect
+			(at 1.59 0 0)
+			(size 1.49 1.73)
+			(layers "F.Cu" "F.Paste" "F.Mask")
+			(net 4 "lv")
+		)
+		(pad "1" smd rect
+			(at -1.59 0 0)
+			(size 1.49 1.73)
+			(layers "F.Cu" "F.Paste" "F.Mask")
+			(net 5 "c_pmid1-1")
+		)
+		(embedded_fonts no)
+		(model "${KIPRJMOD}/../../../parts/blind-power/C1206_L3.2-W1.6-H1.3.step"
+			(offset
+				(xyz 0 0 -0)
+			)
+			(scale
+				(xyz 1 1 1)
+			)
+			(rotate
+				(xyz 0 0 0)
+			)
 		)
 	)
