File: hw/routing/blind-pack-primary/primary-routed.kicad_pcb (KiCad board)
At the start: 2 copper layers, 86 x 104 mm, 54 parts

Commit message: Connect primary battery routing and correct communication protection
Parts:
- moved R12 56.6 mm to (175.8, 197.5)
- moved R8 29.6 mm to (131.8, 202.4), turned to 180 degrees
- moved R4 24.5 mm to (110.5, 199.5)
- moved C7 10.6 mm to (133.8, 200.8), turned to 90 degrees
- moved C8 6.04 mm to (124.7, 202.8), turned to 180 degrees
- moved R9 5.66 mm to (131.8, 197.6), turned to 90 degrees
- moved C5 5.51 mm to (127.8, 203.0), turned to 0 degrees
- moved R2 2.81 mm to (134.0, 197.1)
- moved R3 2.79 mm to (121.0, 202.6), turned to 0 degrees
- moved C6 1.12 mm to (122.5, 198.5), turned to 0 degrees
- moved U1 0.80 mm to (128.0, 199.2)
Connections:
- BT1 pad 2: 2 -> carrier-contact-1
- C1 pad 1: carrier.protection-2 -> 2
- C1 pad 2: 2 -> carrier-contact-1
- C2 pad 1: carrier.protection-2-1 -> carrier.protection-2
- C2 pad 2: carrier.protection-2 -> 2
- C3 pad 2: carrier.protection-2-1 -> carrier.protection-2
- C6 pad 2: 2 -> carrier-contact-1
- C7 pad 2: 2 -> carrier-contact-1
- C8 pad 2: 2 -> carrier-contact-1
- D1 pad 1: ALRT -> carrier-1-2
- D1 pad 2: 2 -> lv
- D2 pad 1: K -> carrier-1-3
- D2 pad 2: 2 -> lv
- D3 pad 1: carrier.protection-K -> carrier-1-4
- D3 pad 2: 2 -> lv
- R1 pad 1: alert_n -> carrier-1-2
- R10 pad 1: carrier-contact-1 -> carrier-1-3
- R10 pad 2: K -> SCL_DOD
- R11 pad 1: carrier-contact-2 -> carrier-1-4
- R11 pad 2: carrier.protection-K -> SDA_DQ
- R13 pad 1: 2 -> carrier-contact-1
- R2 pad 2: 2 -> carrier-contact-1
- R3 pad 2: carrier.protection-2 -> 2
- R4 pad 2: carrier.protection-2-1 -> carrier.protection-2
- R9 pad 2: 2 -> carrier-contact-1
- TP12 pad 1: 2 -> carrier-contact-1
- TP14 pad 1: 2 -> carrier-contact-1
- TP15 pad 1: carrier-contact-3 -> carrier-contact-2
- TP16 pad 1: 2 -> carrier-contact-1
- TP17 pad 1: carrier-contact-4 -> carrier-contact-3
- TP3 pad 1: alert_n -> carrier-1-2
- TP6 pad 1: carrier-contact-1 -> carrier-1-3
- TP7 pad 1: carrier-contact-2 -> carrier-1-4
- U1 pad 10: carrier-contact-3 -> carrier-contact-2
- U1 pad 15: 2 -> carrier-contact-1
- U1 pad 16: carrier-contact-4 -> carrier-contact-3
- U1 pad 18: 2 -> carrier-contact-1
- U1 pad 19: 2 -> carrier-contact-1
- U1 pad 20: 2 -> carrier-contact-1
- U1 pad 21: carrier.protection-2 -> 2
- U1 pad 22: carrier.protection-2 -> 2
- U1 pad 23: carrier.protection-2-1 -> carrier.protection-2
- U1 pad 25: 2 -> carrier-contact-1
- U1 pad 8: K -> SCL_DOD
- U1 pad 9: carrier.protection-K -> SDA_DQ
Routing:
- net carrier-contact-1: track 0.00 -> 344.7 mm, vias 0 -> 11
- net 2: track 153.7 -> 20.8 mm
- net SDA_DQ: track 0.00 -> 114.6 mm, vias 0 -> 10
- net SCL_DOD: track 0.00 -> 112.3 mm, vias 0 -> 6
- net ALRT: track 0.00 -> 109.5 mm, vias 0 -> 8
- net carrier.protection-1: track 0.00 -> 102.5 mm, vias 0 -> 12
- net carrier-contact-2: track 0.00 -> 100.0 mm, vias 0 -> 4
- net carrier-contact-3: track 0.00 -> 92.2 mm, vias 0 -> 6
- net BATTS: track 0.00 -> 80.6 mm, vias 0 -> 8
- net DIS: track 0.00 -> 52.5 mm, vias 0 -> 6
- net contact: track 0.00 -> 51.0 mm
- net carrier-contact: track 0.00 -> 46.3 mm, vias 0 -> 2
- net carrier-1-3: track 0.00 -> 42.0 mm, vias 0 -> 5
- net junction2: track 130.5 -> 166.4 mm
- net carrier-1-4: track 0.00 -> 34.4 mm, vias 0 -> 4
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