File: hw/schematics/blind-carrier/carrier-test.kicad_sch (KiCad schematic)
At the start: 33 parts, among them Q1 AON7400A, Q2 AON7400A, U1 MAX17320G22+

Commit message: Connect primary battery routing and correct communication protection
Connections:
- net ALERT_HOST: now also D1.1 (K)
- net ALRT: no longer D1.1 (K)
- net PACK_GND: now also D1.2 (A), D2.2 (A), D3.2 (A)
- net RAW_GND: no longer D1.2 (A), D2.2 (A), D3.2 (A)
- net SCL_HOST: now also D2.1 (K)
- net SCL_IC: no longer D2.1 (K)
- net SDA_HOST: now also D3.1 (K)
- net SDA_IC: no longer D3.1 (K)
Changed lines of the file:
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@@
 )
   (label
-    "ALRT"
+    "ALERT_HOST"
     (at 90.17 238.76 0)
     (effects
@@
 )
   (label
-    "RAW_GND"
+    "PACK_GND"
     (at 90.17 264.16 0)
     (effects
@@
 )
   (label
-    "SCL_IC"
+    "SCL_HOST"
     (at 363.22 205.74 0)
     (effects
@@
 )
   (label
-    "RAW_GND"
+    "PACK_GND"
     (at 363.22 231.14 0)
     (effects
@@
 )
   (label
-    "SDA_IC"
+    "SDA_HOST"
     (at 254.0 205.74 0)
     (effects
@@
 )
   (label
-    "RAW_GND"
+    "PACK_GND"
     (at 254.0 231.14 0)
     (effects
