File: hw/routing/blind-main/main-routed.kicad_pcb (KiCad board)
At the start: 4 copper layers, 54 x 71 mm, 196 parts

Commit message: Wire monitored USB power into the circuit and owned sensor runtime
Parts:
- removed the C17 at (135.4, 141.8)
- removed the C24 at (103.2, 127.0)
- removed the C32 at (139.4, 147.7)
- removed the R48 at (142.2, 161.9)
- removed the R52 at (127.7, 165.6)
- removed the R56 at (122.6, 160.6)
- removed R64: , blind-control-io:R0402
- removed the R74 at (116.5, 154.0)
- removed the U12 at (149.7, 162.0)
- removed the U15 at (123.0, 134.0)
- added C61: , SAMSUNG_CL10A105KB8NNNC:C0603, F.Cu at (144.0, 166.8)
- added R21: , blind-control-io:R0402, F.Cu at (103.5, 122.7)
- added R35: , UNI_ROYAL_0402WGF1002TCE:R0402, F.Cu at (139.4, 150.2)
- added R38: , UNI_ROYAL_0402WGF1002TCE:R0402, F.Cu at (149.0, 147.9)
- added R53: , UNI_ROYAL_0603WAF1001T5E:R0603, F.Cu at (147.1, 160.6)
- added R60: , UNI_ROYAL_0603WAF1001T5E:R0603, F.Cu at (142.9, 171.0)
- added R66: , UNI_ROYAL_0402WGF3903TCE:R0402, F.Cu at (129.2, 160.8)
- added R73: , blind-regen:R2512, F.Cu at (106.5, 154.0)
- added R78: , blind-control-io:R0402, F.Cu at (104.8, 144.8)
- added U14: , blind-control-io:SOT-363_L2.0-W1.3-P0.65-LS2.1-BR, F.Cu at (122.7, 137.6)
- C17: renamed from J2; footprint blind-harness:CONN-SMD_4P-P1.25_53261-0471 -> SAMSUNG_CL31A106KBHNNNE:C1206
- C24: renamed from R78; footprint blind-control-io:R0402 -> SAMSUNG_CL05B104KB54PNC:C0402
- C32: renamed from R21; footprint blind-control-io:R0402 -> blind-core:C0402
- J2: renamed from U14; footprint blind-control-io:SOT-363_L2.0-W1.3-P0.65-LS2.1-BR -> blind-harness:CONN-SMD_4P-P1.25_53261-0471
- R48: renamed from R85; footprint UNI_ROYAL_0402WGF1002TCE:R0402 -> blind-control-io:R0402
- R52: renamed from R66; footprint UNI_ROYAL_0402WGF3903TCE:R0402 -> blind-usb:R0402
- R56: renamed from R73; footprint blind-regen:R2512 -> blind-power:R0402
- R63: footprint blind-control-io:R0402 -> UNI_ROYAL_0402WGF1002TCE:R0402
- R74: renamed from R35; footprint UNI_ROYAL_0402WGF1002TCE:R0402 -> blind-regen:R2512
- R85: renamed from R60; footprint UNI_ROYAL_0603WAF1001T5E:R0603 -> UNI_ROYAL_0402WGF1002TCE:R0402
- U12: renamed from R53; footprint UNI_ROYAL_0603WAF1001T5E:R0603 -> blind-supervisor:SC-70-6_L2.0-W1.3-P0.65-LS2.1-BR
- U15: renamed from R38; footprint UNI_ROYAL_0402WGF1002TCE:R0402 -> blind-supervisor:SOT-23-6_L2.9-W1.6-P0.95-LS2.8-BR
- moved R85 48.7 mm to (106.0, 139.2)
- moved C32 43.7 mm to (139.4, 147.7), turned to -90 degrees
- moved R48 42.8 mm to (142.2, 161.9)
- moved U15 29.5 mm to (123.0, 134.0)
- moved R74 23.2 mm to (116.5, 154.0), turned to 0 degrees
- moved J2 18.3 mm to (140.0, 131.5), turned to 90 degrees
- moved C24 17.9 mm to (103.2, 127.0), turned to 0 degrees
- moved R56 17.4 mm to (122.6, 160.6), turned to 180 degrees
- moved C17 11.2 mm to (135.4, 141.8)
- moved R63 8.17 mm to (138.0, 162.0)
- moved R52 5.06 mm to (127.7, 165.6), turned to 0 degrees
- moved U12 2.98 mm to (149.7, 162.0), turned to 0 degrees
Connections:
- C17 pad 1: lv -> source-hv
- C17 pad 2: encoder-output-hv -> lv
- C23 pad 1: rail-hv -> host_logic-hv
- C24 pad 1: q_drive-1 -> c_adc-1
- C25 pad 1: rail-hv -> host_logic-hv
- C26 pad 1: rail-hv -> host_logic-hv
- C28 pad 1: rail-hv -> host_logic-hv
- C32 pad 1: controller-1-2 -> CPH
- C32 pad 2: usb_dm -> CPL
- C43 pad 1: rail-hv -> host_logic-hv
- C44 pad 1: rail-hv -> host_logic-hv
- C45 pad 1: rail-hv -> host_logic-hv
- C52 pad 1: rail-hv -> host_logic-hv
- C56 pad 1: rail-hv -> host_logic-hv
- C57 pad 1: rail-hv -> host_logic-hv
- C58 pad 1: rail-hv -> host_logic-hv
- C60 pad 1: rail-hv -> host_logic-hv
- J1 pad 3: pack_sda -> SDA
- J1 pad 4: pack_scl -> SCL
- J2 pad 1: motor_request_n-line -> lv
- J2 pad 2: lv -> encoder-output-hv
- J2 pad 3: heartbeat-line -> channel_a
- J2 pad 4: WDI -> channel_b
- L2 pad 2: rail-hv -> host_logic-hv
- Q2 pad 2: rail-hv -> host_logic-hv
- R19 pad 1: rail-hv -> host_logic-hv
- R20 pad 1: rail-hv -> host_logic-hv
- R22 pad 1: rail-hv -> host_logic-hv
- R24 pad 1: rail-hv -> host_logic-hv
- R26 pad 1: rail-hv -> host_logic-hv
- R27 pad 1: rail-hv -> host_logic-hv
- R27 pad 2: pack_scl -> SCL
- R28 pad 1: rail-hv -> host_logic-hv
- R28 pad 2: pack_sda -> SDA
- R29 pad 1: rail-hv -> host_logic-hv
- R30 pad 1: rail-hv -> host_logic-hv
- R32 pad 1: rail-hv -> host_logic-hv
- R36 pad 1: rail-hv -> host_logic-hv
- R46 pad 1: rail-hv -> host_logic-hv
- R48 pad 1: threshold -> pd-1-1
- R52 pad 1: C -> ILM
- R52 pad 2: r_uv_top1-1 -> lv
- R56 pad 1: hv -> usb-2
- R56 pad 2: r_dump4a-1 -> lv
- R63 pad 1: SCL -> host_logic-hv
- R63 pad 2: lv -> ALERT
- R7 pad 2: rail-hv -> host_logic-hv
- R74 pad 1: rail-hv -> r_dump4a-1
- R74 pad 2: PMODE -> regen-2-1
- R85 pad 1: r_raw_dis1-1 -> threshold
- R85 pad 2: r_raw_dis2-1 -> lv
- R89 pad 1: rail-hv -> host_logic-hv
- R90 pad 1: rail-hv -> host_logic-hv
- R92 pad 1: rail-hv -> host_logic-hv
- R93 pad 1: rail-hv -> host_logic-hv
- U1 pad 14: pack_scl -> SCL
- U1 pad 15: pack_sda -> SDA
- U1 pad 21: INT_n -> ALERT
- U11 pad 22: lv -> host_logic-hv
- U12 pad 1: usb-output-hv -> reset_n
- U12 pad 2: r_out_dis1-1 -> lv
- U15 pad 1: Y -> reset_n
- U16 pad 1: rail-hv -> host_logic-hv
- U16 pad 10: rail-hv -> host_logic-hv
- U17 pad 5: rail-hv -> host_logic-hv
- U2 pad 5: rail-hv -> host_logic-hv
- U3 pad 11: pack_sda -> SDA
- U3 pad 12: pack_scl -> SCL
- U3 pad 2: rail-hv -> host_logic-hv
- U3 pad 24: INT_n -> ALERT
- U8 pad 5: rail-hv -> host_logic-hv
- U9 pad 3: rail-hv -> host_logic-hv
Routing:
- net rail-hv: track 160.8 -> 0.00 mm, vias 12 -> 0
- net host_logic-hv: track 0.00 -> 160.8 mm, vias 0 -> 12
- net lv: track 182.8 -> 178.2 mm, vias 110 -> 108
- net SDA: track 2.09 -> 0.00 mm
- net SCL: track 1.76 -> 0.00 mm
