File: hw/schematics/blind-main/02-charger.kicad_sch (KiCad schematic)
At the start: 36 parts, among them Q1 AO3400A, Q2 MMBT3906LT1G, U1 BQ25798RQMR

Commit message: Wire monitored USB power into the circuit and owned sensor runtime
Connections:
- net CHARGER_IRQ_N renamed POWER_IRQ_N
Changed lines of the file:
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@@
 )
   (global_label
-    "CHARGER_IRQ_N"
+    "POWER_IRQ_N"
     (shape bidirectional)
     (at 124.46 72.39 0)
