File: hw/schematics/blind-main/07-radio.kicad_sch (KiCad schematic)
At the start: 15 parts, among them U3 ESP32-C6-WROOM-1-N4

Commit message: Wire monitored USB power into the circuit and owned sensor runtime
Parts:
- added R63: 10k / SHARED IRQ, UNI_ROYAL_0402WGF1002TCE:R0402, symbol SmartBlinds:P_0402WGF1002TCE
Connections:
- net 3V3: now also R63.1
- net CHARGER_IRQ_N renamed POWER_IRQ_N
- net POWER_IRQ_N: now also R63.2
Other:
- note added: "ESP32-C6. GPIO17 shares PD ALERT + charger INT; one 10k pull-up. SDA/SCL share the single owned 3.3V bus."
- note removed: "ESP32-C6. USB programming shares the USB-C port. Strap-only GPIO4/5/15 are intentionally left open."
Changed lines of the file:
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@@
+  (wire
+    (pts
+      (xy 320.04 219.71)
+      (xy 320.04 227.33))
+    (stroke
+      (width 0)
+      (type default))
+)
+  (global_label
+    "POWER_IRQ_N"
+    (shape bidirectional)
+    (at 320.04 227.33 0)
+    (effects
+      (font
+        (size 1.0 1.0))
+      (justify left))
+)
+  (wire
+    (pts
+      (xy 320.04 209.55)
+      (xy 320.04 201.93))
+    (stroke
+      (width 0)
+      (type default))
+)
+  (global_label
+    "3V3"
+    (shape bidirectional)
+    (at 320.04 201.93 0)
+    (effects
+      (font
+        (size 1.0 1.0))
+      (justify left))
+)
+  (symbol
+    (lib_id "SmartBlinds:P_0402WGF1002TCE")
+    (at 320.04 214.63 270)
+    (unit 1)
+    (in_bom yes)
+    (on_board yes)
+    (dnp no)
+    (property
+      "Reference"
+      "R63"
+      (at 327.66 213.35999999999999 270)
+      (effects
+        (font
+          (size 1.27 1.27))))
+    (property
+      "Value"
+      "10k / SHARED IRQ"
+      (at 327.66 215.89999999999998 270)
+      (effects
+        (font
+          (size 1.27 1.27))))
+    (property
+      "Footprint"
+      "UNI_ROYAL_0402WGF1002TCE:R0402"
+      (at 320.04 214.63 0)
+      (effects
+        (font
+          (size 1.27 1.27))
+        (hide yes)))
+    (property
+      "MPN"
+      "0402WGF1002TCE"
+      (at 320.04 214.63 0)
+      (effects
+        (font
+          (size 1.27 1.27))
+        (hide yes)))
+    (property
+      "LCSC"
+      "C25744"
+      (at 320.04 214.63 0)
+      (effects
+        (font
+          (size 1.27 1.27))
+        (hide yes)))
+    (property
+      "atopile_address"
+      "r_power_irq"
+      (at 320.04 214.63 0)
+      (effects
+        (font
+          (size 1.27 1.27))
+        (hide yes)))
+    (instances
+      (project
+        "smart-blinds-main"
+        (path
+          "/52fe1c56-423a-56fb-97b9-e2338cc62bcc/c9255d8e-68b0-59dc-a1ca-036f9e076650"
+          (reference "R63")
+          (unit 1))))
+    (pin
+      "2"
+)
+    (pin
+      "1"
+))
   (wire
     (pts
@@
 )
   (global_label
-    "CHARGER_IRQ_N"
+    "POWER_IRQ_N"
     (shape bidirectional)
     (at 104.14 101.6 0)
@@
 )
   (text
-    "ESP32-C6. USB programming shares the USB-C port. Strap-only GPIO4/5/15 are intentionally left open."
+    "ESP32-C6. GPIO17 shares PD ALERT + charger INT; one 10k pull-up. SDA/SCL share the single owned 3.3V bus."
     (at 15 26 0)
     (effects
