File: hw/schematics/blind-main/01-usb.kicad_sch (KiCad schematic)
At the start: 33 parts, among them Q3 MMBT3906LT1G, U10 TPS259470LRPWR, U11 STUSB4500QTR

Commit message: Wire monitored USB power into the circuit and owned sensor runtime
Parts:
- removed R63, R64: 100k, blind-control-io:R0402, symbol SmartBlinds:P_0402WGF1003TCE
- added C61: 1u / 50V (VSYS), SAMSUNG_CL10A105KB8NNNC:C0603, symbol SmartBlinds:P_CL10A105KB8NNNC
Connections:
- net GND: now also C61.2; no longer U11.22 (VSYS)
- net POWER_IRQ_N: now reaches U11.19 (ALERT)
- net USB_FACTORY_SCL renamed PACK_SCL
- net USB_FACTORY_SDA renamed PACK_SDA
- new net 3V3: C61.1, U11.22 (VSYS)
- no-connect marks 12 -> 11
Other:
- note added: "32-part unrouted capture. External host logic/pullups and factory access remain open; no physical qualification."
- note added: "Owned MCU I2C at 0x28; VSYS=3.3V. Factory access holds MCU reset, inhibits CE and isolates downstream USB load."
- note removed: "33-part unrouted capture. Native pin equivalence is not PD protocol, ESD/surge or fabrication approval."
- note removed: "Factory NVM required: 5V/1.5A, 9V/2.5A, 15V/2.5A; POWER_ONLY_ABOVE_5V=1. Factory bus is separate from the MCU bus."
Changed lines of the file:
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@@
   (wire
     (pts
+      (xy 144.78 124.46)
+      (xy 144.78 132.08))
+    (stroke
+      (width 0)
+      (type default))
+)
+  (global_label
+    "GND"
+    (shape bidirectional)
+    (at 144.78 132.08 0)
+    (effects
+      (font
+        (size 1.0 1.0))
+      (justify left))
+)
+  (wire
+    (pts
+      (xy 144.78 114.3)
+      (xy 144.78 106.68))
+    (stroke
+      (width 0)
+      (type default))
+)
+  (global_label
+    "3V3"
+    (shape bidirectional)
+    (at 144.78 106.68 0)
+    (effects
+      (font
+        (size 1.0 1.0))
+      (justify left))
+)
+  (symbol
+    (lib_id "SmartBlinds:P_CL10A105KB8NNNC")
+    (at 144.78 119.38 270)
+    (unit 1)
+    (in_bom yes)
+    (on_board yes)
+    (dnp no)
+    (property
+      "Reference"
+      "C61"
+      (at 152.4 118.11 270)
+      (effects
+        (font
+          (size 1.27 1.27))))
+    (property
+      "Value"
+      "1u / 50V (VSYS)"
+      (at 152.4 120.65 270)
+      (effects
+        (font
+          (size 1.27 1.27))))
+    (property
+      "Footprint"
+      "SAMSUNG_CL10A105KB8NNNC:C0603"
+      (at 144.78 119.38 0)
+      (effects
+        (font
+          (size 1.27 1.27))
+        (hide yes)))
+    (property
+      "MPN"
+      "CL10A105KB8NNNC"
+      (at 144.78 119.38 0)
+      (effects
+        (font
+          (size 1.27 1.27))
+        (hide yes)))
+    (property
+      "LCSC"
+      "C15849"
+      (at 144.78 119.38 0)
+      (effects
+        (font
+          (size 1.27 1.27))
+        (hide yes)))
+    (property
+      "atopile_address"
+      "usb.c_vsys"
+      (at 144.78 119.38 0)
+      (effects
+        (font
+          (size 1.27 1.27))
+        (hide yes)))
+    (instances
+      (project
+        "smart-blinds-main"
+        (path
+          "/52fe1c56-423a-56fb-97b9-e2338cc62bcc/4153a6fc-3d10-5549-ba70-3e0a446016e5"
+          (reference "C61")
+          (unit 1))))
+    (pin
+      "2"
+)
+    (pin
+      "1"
+))
+  (wire
+    (pts
       (xy 90.17 157.48)
       (xy 90.17 165.1))
@@
   (wire
     (pts
-      (xy 144.78 124.46)
-      (xy 144.78 132.08))
-    (stroke
-      (width 0)
-      (type default))
-)
-  (global_label
-    "GND"
-    (shape bidirectional)
-    (at 144.78 132.08 0)
-    (effects
-      (font
-        (size 1.0 1.0))
-      (justify left))
-)
-  (wire
-    (pts
-      (xy 144.78 114.3)
-      (xy 144.78 106.68))
-    (stroke
-      (width 0)
-      (type default))
-)
-  (label
-    "USB_FACTORY_SCL"
-    (at 144.78 106.68 0)
-    (effects
-      (font
-        (size 1.0 1.0))
-      (justify left bottom))
-)
-  (symbol
-    (lib_id "SmartBlinds:P_0402WGF1003TCE")
-    (at 144.78 119.38 270)
-    (unit 1)
-    (in_bom yes)
-    (on_board yes)
-    (dnp no)
-    (property
-      "Reference"
-      "R63"
-      (at 152.4 118.11 270)
-      (effects
-        (font
-          (size 1.27 1.27))))
-    (property
-      "Value"
-      "100k"
-      (at 152.4 120.65 270)
-      (effects
-        (font
-          (size 1.27 1.27))))
-    (property
-      "Footprint"
-      "blind-control-io:R0402"
-      (at 144.78 119.38 0)
-      (effects
-        (font
-          (size 1.27 1.27))
-        (hide yes)))
-    (property
-      "MPN"
-      "0402WGF1003TCE"
-      (at 144.78 119.38 0)
-      (effects
-        (font
-          (size 1.27 1.27))
-        (hide yes)))
-    (property
-      "LCSC"
-      "C25741"
-      (at 144.78 119.38 0)
-      (effects
-        (font
-          (size 1.27 1.27))
-        (hide yes)))
-    (property
-      "atopile_address"
-      "usb.r_scl"
-      (at 144.78 119.38 0)
-      (effects
-        (font
-          (size 1.27 1.27))
-        (hide yes)))
-    (instances
-      (project
-        "smart-blinds-main"
-        (path
-          "/52fe1c56-423a-56fb-97b9-e2338cc62bcc/4153a6fc-3d10-5549-ba70-3e0a446016e5"
-          (reference "R63")
-          (unit 1))))
-    (pin
-      "2"
-)
-    (pin
-      "1"
-))
-  (wire
-    (pts
-      (xy 199.39 124.46)
-      (xy 199.39 132.08))
-    (stroke
-      (width 0)
-      (type default))
-)
-  (global_label
-    "GND"
-    (shape bidirectional)
-    (at 199.39 132.08 0)
-    (effects
-      (font
-        (size 1.0 1.0))
-      (justify left))
-)
-  (wire
-    (pts
-      (xy 199.39 114.3)
-      (xy 199.39 106.68))
-    (stroke
-      (width 0)
-      (type default))
-)
-  (label
-    "USB_FACTORY_SDA"
-    (at 199.39 106.68 0)
-    (effects
-      (font
-        (size 1.0 1.0))
-      (justify left bottom))
-)
-  (symbol
-    (lib_id "SmartBlinds:P_0402WGF1003TCE")
-    (at 199.39 119.38 270)
-    (unit 1)
-    (in_bom yes)
-    (on_board yes)
-    (dnp no)
-    (property
-      "Reference"
-      "R64"
-      (at 207.01 118.11 270)
-      (effects
-        (font
-          (size 1.27 1.27))))
-    (property
-      "Value"
-      "100k"
-      (at 207.01 120.65 270)
-      (effects
-        (font
-          (size 1.27 1.27))))
-    (property
-      "Footprint"
-      "blind-control-io:R0402"
-      (at 199.39 119.38 0)
-      (effects
-        (font
-          (size 1.27 1.27))
-        (hide yes)))
-    (property
-      "MPN"
-      "0402WGF1003TCE"
-      (at 199.39 119.38 0)
-      (effects
-        (font
-          (size 1.27 1.27))
-        (hide yes)))
-    (property
-      "LCSC"
-      "C25741"
-      (at 199.39 119.38 0)
-      (effects
-        (font
-          (size 1.27 1.27))
-        (hide yes)))
-    (property
-      "atopile_address"
-      "usb.r_sda"
-      (at 199.39 119.38 0)
-      (effects
-        (font
-          (size 1.27 1.27))
-        (hide yes)))
-    (instances
-      (project
-        "smart-blinds-main"
-        (path
-          "/52fe1c56-423a-56fb-97b9-e2338cc62bcc/4153a6fc-3d10-5549-ba70-3e0a446016e5"
-          (reference "R64")
-          (unit 1))))
-    (pin
-      "2"
-)
-    (pin
-      "1"
-))
-  (wire
-    (pts
       (xy 199.39 190.5)
       (xy 199.39 198.12))
@@
       (type default))
 )
-  (label
-    "USB_FACTORY_SCL"
-    (at 134.62 74.93 0)
+  (global_label
+    "PACK_SCL"
+    (shape bidirectional)
+    (at 134.62 74.93 180)
     (effects
       (font
         (size 1.0 1.0))
-      (justify right bottom))
+      (justify right))
 )
   (wire
@@
       (type default))
 )
-  (label
-    "USB_FACTORY_SDA"
-    (at 134.62 77.47 0)
+  (global_label
+    "PACK_SDA"
+    (shape bidirectional)
+    (at 134.62 77.47 180)
     (effects
       (font
         (size 1.0 1.0))
-      (justify right bottom))
+      (justify right))
 )
   (wire
@@
       (justify left bottom))
 )
-  (no_connect
-    (at 182.88 72.39)
+  (wire
+    (pts
+      (xy 182.88 72.39)
+      (xy 190.5 72.39))
+    (stroke
+      (width 0)
+      (type default))
+)
+  (global_label
+    "POWER_IRQ_N"
+    (shape bidirectional)
+    (at 190.5 72.39 0)
+    (effects
+      (font
+        (size 1.0 1.0))
+      (justify left))
 )
   (no_connect
@@
 )
   (global_label
-    "GND"
+    "3V3"
     (shape bidirectional)
     (at 190.5 64.77 0)
@@
 )
   (text
-    "Factory NVM required: 5V/1.5A, 9V/2.5A, 15V/2.5A; POWER_ONLY_ABOVE_5V=1. Factory bus is separate from the MCU bus."
+    "Owned MCU I2C at 0x28; VSYS=3.3V. Factory access holds MCU reset, inhibits CE and isolates downstream USB load."
     (at 15 24 0)
     (effects
@@
 )
   (text
-    "33-part unrouted capture. Native pin equivalence is not PD protocol, ESD/surge or fabrication approval."
+    "32-part unrouted capture. External host logic/pullups and factory access remain open; no physical qualification."
     (at 15 281 0)
     (effects

Commit message: Make the cleaner controller reproducible from circuit source (#3)
* Rebuild cleaner controller from circuit source and verify native previews

* Use compiler-compatible Python without changing native render runtime
Parts:
- added C62: 47n / 50V, blind-power:C0402, symbol SmartBlinds:P_0402B473K500NT
- added C63: 4.7u / 50V, blind-usb:C1206, symbol SmartBlinds:P_CL31A475KBHNNNE
- added R64: 1.2k, blind-core:R0402, symbol SmartBlinds:P_0402WGF1201TCE
- added R94: 402k, blind-usb-protection:R0402, symbol SmartBlinds:P_0402WGF4023TCE
- added R95: 30.1k / 0.1%, blind-usb-protection:R0402, symbol SmartBlinds:P_RT0402BRD0730K1L
- added R96: 390k, UNI_ROYAL_0402WGF3903TCE:R0402, symbol SmartBlinds:P_0402WGF3903TCE
- added R97: 100k, blind-control-io:R0402, symbol SmartBlinds:P_0402WGF1003TCE
- added R98: 4.7k, blind-control-io:R0402, symbol SmartBlinds:P_0402WGF4701TCE
- added U18: TPS26600PWPR, blind-usb-protection:TPS26600_PWP16, symbol SmartBlinds:P_TPS26600PWPR
- added U19: TVS1800DRVR, blind-usb-protection:TVS1800_DRV6, symbol SmartBlinds:P_TVS1800DRVR
Connections:
- net GND: now also C63.2, R97.2, U18.9 (GND), U19.1 (GND), U19.2 (GND), U19.3 (GND), U19.7 (GND)
- net USB_VBUS_RAW renamed USB_GUARDED
- net USB_GUARDED: now also C63.1, R97.1, U18.15 (OUT), U18.16 (OUT), U19.4 (IN), U19.5 (IN), U19.6 (IN); no longer C49.1, D5.1 (K), USBC1.A4B9 (VBUS), USBC1.B4A9 (VBUS)
- new net USB_CUT_ILIM: R64.1, U18.11 (ILIM)
- new net USB_CUT_ILIM_MID: R64.2, R98.1
- new net USB_CUT_MODE: R94.1, U18.6 (MODE)
- new net USB_CUT_OVP: R95.1, R96.2, U18.5 (OVP)
- new net USB_CUT_RTN: C62.2, R94.2, R95.2, R98.2, U18.17 (EP), U18.8 (RTN)
- new net USB_CUT_SLEW: C62.1, U18.12 (dVdT)
- new net USB_RAW: C49.1, D5.1 (K), R96.1, U18.1 (IN), U18.2 (IN), U18.3 (UVLO), USBC1.A4B9 (VBUS), USBC1.B4A9 (VBUS)
- no-connect marks 11 -> 16
Other:
- note added: "42-part source capture with upstream cutoff. Routing, factory access and physical qualification remain incomplete."
- note removed: "32-part unrouted capture. External host logic/pullups and factory access remain open; no physical qualification."
