File: hw/schematics/blind-main/smart-blinds-main.kicad_sch (KiCad schematic)
At the start: 0 parts

Commit message: Wire monitored USB power into the circuit and owned sensor runtime
Other:
- note added: "16 parts / 70 pin identities"
- note added: "32 parts / 111 pin identities"
- note removed: "15 parts / 68 pin identities"
- note removed: "33 parts / 113 pin identities"
Changed lines of the file:
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@@
           (page "2")))))
   (text
-    "33 parts / 113 pin identities"
+    "32 parts / 111 pin identities"
     (at 24 56 0)
     (effects
@@
           (page "8")))))
   (text
-    "15 parts / 68 pin identities"
+    "16 parts / 70 pin identities"
     (at 24 126 0)
     (effects

Commit message: Make the cleaner controller reproducible from circuit source (#3)
* Rebuild cleaner controller from circuit source and verify native previews

* Use compiler-compatible Python without changing native render runtime
Other:
- note added: "206 circuit features. USB-C charging, protected pack input, radio, motor and local controls."
- note added: "42 parts / 151 pin identities"
- note removed: "196 circuit features. USB-C charging, protected pack input, radio, motor and local controls."
- note removed: "32 parts / 111 pin identities"
Changed lines of the file:
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@@
           (page "2")))))
   (text
-    "32 parts / 111 pin identities"
+    "42 parts / 151 pin identities"
     (at 24 56 0)
     (effects
@@
 )
   (text
-    "196 circuit features. USB-C charging, protected pack input, radio, motor and local controls."
+    "206 circuit features. USB-C charging, protected pack input, radio, motor and local controls."
     (at 15 26 0)
     (effects
