File: hw/layouts/blind-carrier/carrier-test/carrier-test.kicad_pcb (KiCad board)
At the start: 2 copper layers, 33 parts

Commit message: Connect primary battery routing and correct communication protection
Connections:
- D1 pad 1: ALRT -> alert_n
- D1 pad 2: lv -> pack-lv
- D2 pad 1: K -> scl
- D2 pad 2: lv -> pack-lv
- D3 pad 1: carrier-K -> sda
- D3 pad 2: lv -> pack-lv
- R10 pad 2: K -> SCL_DOD
- R11 pad 2: carrier-K -> SDA_DQ
- U1 pad 8: K -> SCL_DOD
- U1 pad 9: carrier-K -> SDA_DQ
Changed lines of the file:
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@@
 	(net 21 "ZVC")
 	(net 22 "ALRT")
-	(net 23 "alert_n")
 	(net 24 "AOLDO")
 	(net 26 "2")
@@
 	(net 30 "PCKP")
 	(net 31 "PFAIL")
-	(net 32 "scl")
-	(net 33 "sda")
 	(net 34 "1")
-	(net 35 "K")
-	(net 36 "carrier-K")
+	(net 35 "SCL_DOD")
+	(net 36 "SDA_DQ")
 	(net 39 "hv")
 	(net 40 "cell1b-hv")
@@
 	(net 44 "cell3a-hv")
 	(net 45 "cell3b-hv")
-	(net 46 "pack-lv")
 	(net 47 "cell2b-lv")
 	(net 48 "carrier-2-1")
@@
 	(net 5 "carrier-G")
 	(net 6 "pack-hv")
+	(net 4 "alert_n")
+	(net 7 "sda")
+	(net 8 "pack-lv")
+	(net 9 "scl")
 	(footprint "blind-carrier:FUSE-SMD_L6.1-W2.7"
 		(layer "F.Cu")
@@
 			(size 0.665 0.28)
 			(layers "F.Cu" "F.Mask" "F.Paste")
-			(net 35 "K")
+			(net 35 "SCL_DOD")
 		)
 		(pad "9" smd rect
@@
 			(size 0.665 0.28)
 			(layers "F.Cu" "F.Mask" "F.Paste")
-			(net 36 "carrier-K")
+			(net 36 "SDA_DQ")
 		)
 		(pad "10" smd rect
@@
 			(size 0.28 0.665)
 			(layers "F.Cu" "F.Mask" "F.Paste")
-			(net 46 "pack-lv")
+			(net 8 "pack-lv")
 		)
 		(pad "15" smd rect
@@
 			(size 1.65 3.68)
 			(layers "F.Cu" "F.Mask" "F.Paste")
-			(net 46 "pack-lv")
+			(net 8 "pack-lv")
 		)
 		(embedded_fonts no)
@@
 			(size 0.566 0.54)
 			(layers "F.Cu" "F.Mask" "F.Paste")
-			(net 33 "sda")
+			(net 7 "sda")
 		)
 		(pad "2" smd rect
@@
 			(size 0.566 0.54)
 			(layers "F.Cu" "F.Mask" "F.Paste")
-			(net 36 "carrier-K")
+			(net 36 "SDA_DQ")
 		)
 		(embedded_fonts no)
@@
 			(size 0.95 1.15)
 			(layers "F.Cu" "F.Mask" "F.Paste")
-			(net 36 "carrier-K")
+			(net 7 "sda")
 		)
 		(pad "2" smd rect
@@
 			(size 0.95 1.15)
 			(layers "F.Cu" "F.Mask" "F.Paste")
-			(net 17 "lv")
+			(net 8 "pack-lv")
 		)
 		(embedded_fonts no)
@@
 			(size 0.566 0.54)
 			(layers "F.Cu" "F.Mask" "F.Paste")
-			(net 32 "scl")
+			(net 9 "scl")
 		)
 		(pad "2" smd rect
@@
 			(size 0.566 0.54)
 			(layers "F.Cu" "F.Mask" "F.Paste")
-			(net 35 "K")
+			(net 35 "SCL_DOD")
 		)
 		(embedded_fonts no)
@@
 			(size 0.95 1.15)
 			(layers "F.Cu" "F.Mask" "F.Paste")
-			(net 35 "K")
+			(net 9 "scl")
 		)
 		(pad "2" smd rect
@@
 			(size 0.95 1.15)
 			(layers "F.Cu" "F.Mask" "F.Paste")
-			(net 17 "lv")
+			(net 8 "pack-lv")
 		)
 		(embedded_fonts no)
@@
 			(size 0.566 0.54)
 			(layers "F.Cu" "F.Mask" "F.Paste")
-			(net 23 "alert_n")
+			(net 4 "alert_n")
 		)
 		(pad "2" smd rect
@@
 			(size 0.95 1.15)
 			(layers "F.Cu" "F.Mask" "F.Paste")
-			(net 22 "ALRT")
+			(net 4 "alert_n")
 		)
 		(pad "2" smd rect
@@
 			(size 0.95 1.15)
 			(layers "F.Cu" "F.Mask" "F.Paste")
-			(net 17 "lv")
+			(net 8 "pack-lv")
 		)
 		(embedded_fonts no)
