File: hw/layouts/blind-usb/usb-test/usb-test.kicad_pcb (KiCad board)
At the start: 2 copper layers, 33 parts

Commit message: Correct USB connector lands and document PD factory policy evidence
Parts:
- USBC1: footprint UNKNOWN_TYPE_C_31_M_12:USB-C_SMD-TYPE-C-31-M-12_1 -> blind-usb:HRO_TYPE_C_31_M_12

Commit message: Wire monitored USB power into the circuit and owned sensor runtime
Parts:
- removed R17, R18: , blind-control-io:R0402
- added C6: , SAMSUNG_CL10A105KB8NNNC:C0603, F.Cu at (0.00, 0.00)
Connections:
- C3 pad 1: hv -> raw-hv
- D1 pad 2: hv -> raw-hv
- D3 pad 1: hv -> raw-hv
- Q1 pad 2: hv -> raw-hv
- R11 pad 1: hv -> raw-hv
- R13 pad 1: hv -> raw-hv
- R5 pad 1: hv -> raw-hv
- U1 pad 5: hv -> raw-hv
- U2 pad 22: lv -> hv
- USBC1 pad A4B9: hv -> raw-hv
- USBC1 pad B4A9: hv -> raw-hv

Commit message: Make the cleaner controller reproducible from circuit source (#3)
* Rebuild cleaner controller from circuit source and verify native previews

* Use compiler-compatible Python without changing native render runtime
Parts:
- added C7: , blind-power:C0402, F.Cu at (50.0, 0.00)
- added C8: , blind-usb:C1206, F.Cu at (60.0, 0.00)
- added R17: , blind-core:R0402, F.Cu at (30.0, 0.00)
- added R18: , blind-usb-protection:R0402, F.Cu at (40.0, 0.00)
- added R22: , blind-usb-protection:R0402, F.Cu at (20.0, 0.00)
- added R23: , UNI_ROYAL_0402WGF3903TCE:R0402, F.Cu at (10.0, 0.00)
- added R24: , blind-control-io:R0402, F.Cu at (70.0, 0.00)
- added R25: , blind-control-io:R0402, F.Cu at (0.00, 0.00)
- added U3: , blind-usb-protection:TPS26600_PWP16, F.Cu at (0.00, 0.00)
- added U4: , blind-usb-protection:TVS1800_DRV6, F.Cu at (80.0, 0.00)
Connections:
- net 2 renamed usb-2
- net DVDT renamed usb-DVDT
- D1 pad 2: raw-hv -> guarded-hv
- Q1 pad 2: raw-hv -> guarded-hv
- R11 pad 1: raw-hv -> guarded-hv
- R11 pad 2: usb-1-10 -> usb-1-11
- R12 pad 1: usb-1-10 -> usb-1-11
- R13 pad 1: raw-hv -> guarded-hv
- R13 pad 2: usb-1-11 -> usb-1-12
- R14 pad 1: usb-1-11 -> usb-1-12
- R14 pad 2: usb-1-12 -> usb-1-13
- R15 pad 1: usb-1-12 -> usb-1-13
- R20 pad 2: usb-1-13 -> usb-1-14
- R21 pad 1: usb-1-13 -> usb-1-14
- R5 pad 1: raw-hv -> guarded-hv
- R7 pad 2: usb-1-8 -> usb-1-9
- R8 pad 1: usb-1-8 -> usb-1-9
- R8 pad 2: usb-1-9 -> usb-1-10
- R9 pad 1: usb-1-9 -> usb-1-10
- U1 pad 5: raw-hv -> guarded-hv
